File: cc3220modasf.sch (KiCad schematic (older format))
At the start: 90 parts, among them J1 Conn_02x05_Odd_Even, J10 Conn_01x02, J11 Conn_02x04_Odd_Even, J13 Conn_02x05_Counter_Clockwise, J14 Conn_01x02, J15 Conn_01x02, J2 Conn_02x05_Odd_Even, J22 Conn_02x04_Odd_Even, J26 Conn_01x03, J3 Conn_01x06, J5 Conn_01x03, J6 Conn_01x03, Q4 BSS138, Q5 TP0610T, Q6 BSS138, Q7 BSS138, SW2 SW_DIP_x01, U10 TMP006AIYZFR, U7 OPA4340UA, U9 CC3220MODASF12MONR

Commit message: Changed U10 to TMP116AIDRVR. Added new sybmol/footprint bom, pos files and README into repo.
Parts:
- removed R114, R119, R121, R126, R127, R132, R133: 0, Resistor_SMD:R_0402_1005Metric, symbol Device:R_Small
- removed U10: TMP006AIYZFR, TMP006AIYZFR:TMP006AIYZFR, symbol cc3220modasf:TMP006AIYZFR
- added R116, R117, R118: 4k87, Resistor_SMD:R_0603_1608Metric, symbol Device:R_Small
- added U10: TMP116AIDRVR, TMP116:TMP116AIDRVR, symbol tmp116:TMP116AIDRVR
- D10: value LED -> RED LED
- D4, D5: MFG Part Num CD0603-B00340 -> CD0603-B0240R/B00340
- D8: value LED -> GREEN LED
- D9: value LED -> YELLOW LED
- J1, J2: MFG Name (none) -> Samtec Inc; MFG Part Num (none) -> TSW-105-15-G-D
- Q5: value TP0610T -> FDN358P
- R107: value 270 -> 270R; footprint Resistor_SMD:R_0402_1005Metric -> Resistor_SMD:R_0603_1608Metric; MFG Name Panasonic -> Vishay-Dale; MFG Part Num ERJ-2GE0R00X -> CRCW0603270RJNEA
- R136: MFG Part Num CRCW04021K00JNED -> CRCW04021K00JNEDC
- R139: MFG Part Num CRCW040210K0JNED -> CRCW040210K0JNEDC
- R145, R146, R147: value 270 -> 270R; MFG Part Num CRCW0603270RJNEA -> CRCW0603270RJNEAC
- R149, R150, R151: MFG Part Num CRCW0402100KJNED -> CRCW0402100KJNEDC
- R84, R87, R92, R93: value 470 -> 470R
- U9: MFG Name (none) -> Texas Instruments; MFG Part Num (none) -> CC3220MODASF12MON
Connections:
- wire segments 127 -> 126
- no-connect marks 21 -> 20
Other:
- moved on the sheet: J14, J15
